File: v1/superbatt/superbatt.kicad_pcb (KiCad board)
At the start: 2 copper layers, 47.2 x 47.2 mm, 14 parts, among them J1 Screw_Terminal_01x02, J2 Conn_01x02_Socket, J3 USB_B_Micro, J4 Screw_Terminal_01x02, J5 Conn_01x02_Socket

Commit message: update
Parts:
- removed J2, J5: Conn_01x02_Socket, Connector_PinHeader_2.54mm:PinHeader_1x02_P2.54mm_Vertical
- added J6: Conn_01x04_Socket, Connector_PinSocket_2.54mm:PinSocket_1x04_P2.54mm_Vertical, F.Cu at (16.2, 41.8)
- C2: footprint Capacitor_THT:CP_Radial_D13.0mm_P5.00mm -> superbatt:CP_Radial_D22.0mm_P5.00mm_SnapIn
- R1: footprint Resistor_THT:R_Axial_DIN0309_L9.0mm_D3.2mm_P12.70mm_Horizontal -> Resistor_THT:R_Axial_DIN0207_L6.3mm_D2.5mm_P10.16mm_Horizontal
- moved D3 27.5 mm to (10.5, 34.2)
- moved D1 25.8 mm to (40.7, 34.4), turned to 180 degrees
- moved R1 16.7 mm to (9.64, 9.40), turned to 0 degrees
- moved D2 15.8 mm to (37.7, 9.40)
- moved C2 2.94 mm to (15.7, 22.8)
- moved J4 2.82 mm to (1.60, 20.5)
- moved J1 2.81 mm to (38.8, 25.6)
- moved J3 0.55 mm to (0.15, 8.53)
Routing:
- net GND: track 122.2 -> 0.00 mm, vias 10 -> 0
- net Net-(D1-K): track 100.4 -> 0.00 mm, vias 7 -> 0
- net Net-(D2-A): track 70.3 -> 0.00 mm, vias 5 -> 0
- net Net-(D3-A): track 19.1 -> 0.00 mm, vias 1 -> 0
- net unconnected-(J3-Shield-Pad6): track 15.5 -> 0.00 mm
- net Net-(D2-K): track 9.60 -> 0.00 mm
Other:
- board text added: "Design files & guides:"
- board text removed: "Design files & guide:"
- board text removed: "VIN (5V Max)"

Commit message: update
Parts:
- moved R1 18.4 mm to (28.0, 9.20)
- moved D2 18.0 mm to (19.7, 9.20)
Routing:
- net GND: track 0.00 -> 81.2 mm, vias 0 -> 4
- net Net-(D1-K): track 0.00 -> 74.2 mm, vias 0 -> 5
- net Net-(D2-A): track 0.00 -> 47.9 mm, vias 0 -> 3
- net Net-(D2-K): track 0.00 -> 42.6 mm, vias 0 -> 2
- net Net-(D3-A): track 0.00 -> 22.1 mm, vias 0 -> 2
- net unconnected-(J3-Shield-Pad6): track 0.00 -> 15.5 mm
